File: coaster_backboard/coaster_backboard.kicad_sch (KiCad schematic)
At the start: 127 parts, among them J1 USB, J2 MP, J3 MP, J4 MP, J5 MP, J6 Solderpad, J7 Solderpad, J8 USB, P1 TC2030, U1 STM32F072C8Tx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

Commit message: updated schematic
Other:
- note added: "Pink: https://jlcpcb.com/partdetail/Xinglight-XL_1608UPC06/C2977076 Blue (Cyan): https://jlcpcb.com/partdetail/Meihua-MHT192WDTICE/C389522 RGB: https://jlcpcb.com/partdetail/169447-FC_B1010RGBTHG/C158099 For the LEDs labelled "white", replace them with colours of your choice that represent the night sky as you like it! I used: 8 white LEDs: https://jlcpcb.com/partdetail/85434-NCD0603W1/C84265 3 C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"
