File: coaster_frontboard/coaster_frontboard.sch (KiCad schematic (older format))
At the start: 3 parts

Commit message: updated hw
Parts:
- added J1: NTC, TestPoint:TestPoint_Pad_D1.5mm, symbol Connector:Conn_01x01_Female
- added J2: GND, TestPoint:TestPoint_Pad_D1.5mm, symbol Connector:Conn_01x01_Female
- added J3, J4, J5, J6: MP, TestPoint:TestPoint_Pad_D1.5mm, symbol Connector:Conn_01x01_Female
- added TH1: NTC, otter:R_0402, symbol Device:Thermistor_NTC
Connections:
- new net: J2.1 (Pin_1), TH1.1
- new net: J1.1 (Pin_1), TH1.2
- no-connect marks 0 -> 4
Changed lines of the file:
@@
 	1    0    0    -1
 $EndComp
+$Comp
+L Connector:Conn_01x01_Female J2
+U 1 1 6398F814
+P 6050 3350
+F 0 "J2" H 6078 3376 50  0000 L CNN
+F 1 "GND" H 6078 3285 50  0000 L CNN
+F 2 "TestPoint:TestPoint_Pad_D1.5mm" H 6050 3350 50  0001 C CNN
+F 3 "~" H 6050 3350 50  0001 C CNN
+	1    6050 3350
+	1    0    0    -1
+$EndComp
+$Comp
+L Device:Thermistor_NTC TH1
+U 1 1 6398FA96
+P 5700 3350
+F 0 "TH1" V 5410 3350 50  0000 C CNN
+F 1 "NTC" V 5501 3350 50  0000 C CNN
+F 2 "otter:R_0402" H 5700 3400 50  0001 C CNN
+F 3 "~" H 5700 3400 50  0001 C CNN
+	1    5700 3350
+	0    1    1    0
+$EndComp
+$Comp
+L Connector:Conn_01x01_Female J1
+U 1 1 639904D2
+P 5350 3350
+F 0 "J1" H 5378 3284 50  0000 L CNN
+F 1 "NTC" H 5378 3375 50  0000 L CNN
+F 2 "TestPoint:TestPoint_Pad_D1.5mm" H 5350 3350 50  0001 C CNN
+F 3 "~" H 5350 3350 50  0001 C CNN
+	1    5350 3350
+	-1   0    0    1
+$EndComp
+$Comp
+L Connector:Conn_01x01_Female J3
+U 1 1 639916F5
+P 6250 2000
+F 0 "J3" H 6278 2026 50  0000 L CNN
+F 1 "MP" H 6278 1935 50  0000 L CNN
+F 2 "TestPoint:TestPoint_Pad_D1.5mm" H 6250 2000 50  0001 C CNN
+F 3 "~" H 6250 2000 50  0001 C CNN
+	1    6250 2000
+	1    0    0    -1
+$EndComp
+NoConn ~ 6050 2000
+$Comp
+L Connector:Conn_01x01_Female J4
+U 1 1 63991A5F
+P 6250 2150
+F 0 "J4" H 6278 2176 50  0000 L CNN
+F 1 "MP" H 6278 2085 50  0000 L CNN
+F 2 "TestPoint:TestPoint_Pad_D1.5mm" H 6250 2150 50  0001 C CNN
+F 3 "~" H 6250 2150 50  0001 C CNN
+	1    6250 2150
+	1    0    0    -1
+$EndComp
+NoConn ~ 6050 2150
+$Comp
+L Connector:Conn_01x01_Female J5
+U 1 1 63991D2D
+P 6250 2300
+F 0 "J5" H 6278 2326 50  0000 L CNN
+F 1 "MP" H 6278 2235 50  0000 L CNN
+F 2 "TestPoint:TestPoint_Pad_D1.5mm" H 6250 2300 50  0001 C CNN
+F 3 "~" H 6250 2300 50  0001 C CNN
+	1    6250 2300
+	1    0    0    -1
+$EndComp
+NoConn ~ 6050 2300
+$Comp
+L Connector:Conn_01x01_Female J6
+U 1 1 63991F87
+P 6250 2450
+F 0 "J6" H 6278 2476 50  0000 L CNN
+F 1 "MP" H 6278 2385 50  0000 L CNN
+F 2 "TestPoint:TestPoint_Pad_D1.5mm" H 6250 2450 50  0001 C CNN
+F 3 "~" H 6250 2450 50  0001 C CNN
+	1    6250 2450
+	1    0    0    -1
+$EndComp
+NoConn ~ 6050 2450
 $EndSCHEMATC
