File: coaster_frontboard/coaster_frontboard.kicad_pcb (KiCad board)
At the start: 2 copper layers, 93 x 93 mm, 3 parts

Commit message: updated hw
Parts:
- added G***: LOGO, otter:stars_kani_aji_bmask, F.Cu at (116.6, 71.2)
- added G***: LOGO, otter:shark_girl_kani_aji_bmask, F.Cu at (76.0, 100.8)
- added J1: NTC, TestPoint:TestPoint_Pad_D1.5mm, B.Cu at (76.8, 65.2)
- added J2: GND, TestPoint:TestPoint_Pad_D1.5mm, B.Cu at (74.0, 65.2)
- added J3: MP, TestPoint:TestPoint_Pad_D1.5mm, B.Cu at (90.0, 96.5)
- added J4: MP, TestPoint:TestPoint_Pad_D1.5mm, B.Cu at (59.5, 59.5)
- added J5: MP, TestPoint:TestPoint_Pad_D1.5mm, B.Cu at (133.5, 133.5)
- added J6: MP, TestPoint:TestPoint_Pad_D1.5mm, B.Cu at (137.5, 55.5)
- added TH1: NTC, otter:R_0402, B.Cu at (83.9, 75.3)
Routing:
- net Net-(J2-Pad1): track 0.00 -> 14.0 mm
- net Net-(J1-Pad1): track 0.00 -> 13.2 mm
Other:
- board text removed: "TODO ARTWORK AUF ALLE LAYER"

Commit message: updated frontboard
Other:
- net class Default removed
